File: fe11_usbhub_tryout.sch (KiCad schematic (older format))
At the start: 0 parts

Commit message: update,
Parts:
- added U?: FE1.1_LQFP48, footprint-lib:FE1.1_LQFP48, symbol taobao-components:FE1.1_LQFP48

Commit message: update,
Parts:
- added C? (x2): C10pf,0603, Capacitor_SMD:C_0603_1608Metric_Pad1.05x0.95mm_HandSolder, symbol taobao-c:C10pf,0603
- added C? (x2): C106,0603, Capacitor_SMD:C_0603_1608Metric_Pad1.05x0.95mm_HandSolder, symbol taobao-c:C106,0603
- added D? (x4): LED_dual_small, symbol taobao-components:LED_dual_small
- added D?: LED_GREEN,0603, footprint-lib:LED_0603_1608Metric, symbol taobao-led:LED_GREEN,0603
- added J? (x5): USB_HEADER, footprint-lib:USB_DEBUG, symbol taobao-components:USB_HEADER
- added R? (x4): R101,0603, Resistor_SMD:R_0603_1608Metric_Pad1.05x0.95mm_HandSolder, symbol taobao-r:R101,0603
- added R?: R103,0603, Resistor_SMD:R_0603_1608Metric_Pad1.05x0.95mm_HandSolder, symbol taobao-r:R103,0603
- added R?: R272,0603, Resistor_SMD:R_0603_1608Metric_Pad1.05x0.95mm_HandSolder, symbol taobao-r:R272,0603
- added RN?: R_Pack04, symbol Device:R_Pack04
- added TP?: 1V8_ref, symbol Connector:TestPoint
- added TP?: 3V3_ref, symbol Connector:TestPoint
- added U? (x2): MIC2026, footprint-lib:MIC2026_SOIC8, symbol taobao-components:MIC2026
- added Y?: O_12M,3225, footprint-lib:OSC_3225, symbol taobao-osc:O_12M,3225
Connections:
- net labels added: +3V3, +5V, GND
- wire segments 0 -> 163
Other:
- moved on the sheet: U?

Commit message: update,
Parts:
- removed R? (x4): R101,0603, Resistor_SMD:R_0603_1608Metric_Pad1.05x0.95mm_HandSolder, symbol taobao-r:R101,0603
- added RN?: R_Pack04, symbol Device:R_Pack04
Connections:
- net labels added: USB_3V3, VBUS_A, VBUS_B, VBUS_C, VBUS_D
- net labels removed: +3V3
- wire segments 163 -> 175
Other:
- moved on the sheet: D?

Commit message: update,
Parts:
- added C4, C6: C104,0603, Capacitor_SMD:C_0603_1608Metric_Pad1.05x0.95mm_HandSolder, symbol taobao-c:C106,0603
- added R1, R2: R104,0603, Resistor_SMD:R_0603_1608Metric_Pad1.05x0.95mm_HandSolder, symbol taobao-r:R104,0603
- gave numbers to parts that had none: 24
Connections:
- net GND: now also J1.GND, J2.GND, J3.GND, J4.GND, J5.GND, U1.37 (DIS_REG), C4.2, C6.2
- net HUB_1V8: now reaches C5.1, TP1.1, U1.26 (VREG18), U1.29 (VD18), U1.3 (VD18), U1.9 (VD_PLL_1V8)
- net HUB_1V8: now also C6.1
- net at U1.34 (XRSTJ): now also R2.2
- net at U1.35 (VBUSM): now also R1.2
- net at U1.42 (DRV): now also D1.1 (K2), D1.2 (A2), D2.1 (K2), D2.2 (A2), D3.1 (K2), D3.2 (A2), D4.1 (K2), D4.2 (A2), D5.2 (A)
- net USB_3V3 renamed HUB_3V3
- net HUB_3V3: now also C4.1, R1.1, R2.1
- no-connect marks 0 -> 3
Other:
- moved on the sheet: C3, C5, TP2

Commit message: update,
Parts:
- added C? (x4): CP100uf,10V, Capacitor_SMD:CP_Elec_6.3x5.3, symbol taobao-cp:CP100uf,10V
- added C? (x4): C104,0603, Capacitor_SMD:C_0603_1608Metric_Pad1.05x0.95mm_HandSolder, symbol taobao-c:C104,0603
- added R?: R104,0603, Resistor_SMD:R_0603_1608Metric_Pad1.05x0.95mm_HandSolder, symbol taobao-r:R104,0603
Connections:
- net GND: now also C?.2, C?.2, C?.2, C?.2, C?.2, C?.2, C?.2, C?.2
- net HUB_3V3: now also R?.1
- net VBUS_A: now also C?.1, C?.1
- net VBUS_B: now also C?.1, C?.1
- net VBUS_C: now also C?.1, C?.1
- net VBUS_D: now also C?.1, C?.1
- net at U1.36 (BUS_B): now also R?.2
- new net: D1.1 (K2), D1.2 (A2), D2.1 (K2), D2.2 (A2), D3.1 (K2), D3.2 (A2), D4.1 (K2), D4.2 (A2), D5.2 (A), U1.42 (DRV)
- no-connect marks 3 -> 1
Other:
- moved on the sheet: J1, J5

Commit message: update footprint,
Parts:
- gave numbers to parts that had none: 9
Connections:
- new net: D1.1 (K2), D1.2 (A2), D2.1 (K2), D2.2 (A2), D3.1 (K2), D3.2 (A2), D4.1 (K2), D4.2 (A2), D5.2 (A), U1.42 (DRV)
Changed lines of the file:
@@
 	3850 5750 3950 5750
 $Comp
-L taobao-components:HUB_3V3 #PWR?
+L taobao-components:HUB_3V3 #PWR0103
 U 1 1 5D3F54CA
 P 3500 5650
-F 0 "#PWR?" H 3500 5500 50  0001 C CNN
+F 0 "#PWR0103" H 3500 5500 50  0001 C CNN
 F 1 "HUB_3V3" H 3500 5750 50  0000 C CNN
 F 2 "" H 3500 5650 50  0001 C CNN
@@
 	3500 5750 3850 5750
 $Comp
-L taobao-components:HUB_3V3 #PWR?
+L taobao-components:HUB_3V3 #PWR0104
 U 1 1 5CF0133F
 P 6900 6250
-F 0 "#PWR?" H 6900 6100 50  0001 C CNN
+F 0 "#PWR0104" H 6900 6100 50  0001 C CNN
 F 1 "HUB_3V3" H 6900 6350 50  0000 C CNN
 F 2 "" H 6900 6250 50  0001 C CNN
@@
 $EndComp
 $Comp
-L taobao-r:R104,0603 R?
+L taobao-r:R104,0603 R5
 U 1 1 5CF01349
 P 6700 6250
-F 0 "R?" H 6600 6300 50  0000 R CNN
+F 0 "R5" H 6600 6300 50  0000 R CNN
 F 1 "R104,0603" H 6600 6250 50  0000 R CNN
 F 2 "Resistor_SMD:R_0603_1608Metric_Pad1.05x0.95mm_HandSolder" H 6700 6250 50  0001 C CNN
@@
 	10750 6000 10500 6000
 $Comp
-L taobao-cp:CP100uf,10V C?
+L taobao-cp:CP100uf,10V C13
 U 1 1 5CF1C676
 P 10250 6200
-F 0 "C?" H 10150 6250 50  0000 R CNN
+F 0 "C13" H 10150 6250 50  0000 R CNN
 F 1 "CP100uf,10V" H 10150 6200 50  0000 R CNN
 F 2 "Capacitor_SMD:CP_Elec_6.3x5.3" H 10250 6200 50  0001 C CNN
@@
 $EndComp
 $Comp
-L taobao-c:C104,0603 C?
+L taobao-c:C104,0603 C14
 U 1 1 5CF1D0EE
 P 10500 6200
-F 0 "C?" H 10600 6250 50  0000 L CNN
+F 0 "C14" H 10600 6250 50  0000 L CNN
 F 1 "C104,0603" H 10600 6200 50  0000 L CNN
 F 2 "Capacitor_SMD:C_0603_1608Metric_Pad1.05x0.95mm_HandSolder" H 10500 6200 50  0001 C CNN
@@
 	10500 6000 10250 6000
 $Comp
-L power:GND #PWR?
+L power:GND #PWR0105
 U 1 1 5CF36FE0
 P 10250 6400
-F 0 "#PWR?" H 10250 6150 50  0001 C CNN
+F 0 "#PWR0105" H 10250 6150 50  0001 C CNN
 F 1 "GND" H 10300 6200 50  0000 C CNN
 F 2 "" H 10250 6400 50  0001 C CNN
@@
 	10250 6300 10250 6400
 $Comp
-L power:GND #PWR?
+L power:GND #PWR0106
 U 1 1 5CF4400E
 P 10500 6400
-F 0 "#PWR?" H 10500 6150 50  0001 C CNN
+F 0 "#PWR0106" H 10500 6150 50  0001 C CNN
 F 1 "GND" H 10550 6200 50  0000 C CNN
 F 2 "" H 10500 6400 50  0001 C CNN
@@
 	10750 5200 10500 5200
 $Comp
-L taobao-cp:CP100uf,10V C?
+L taobao-cp:CP100uf,10V C11
 U 1 1 5CF510E2
 P 10250 5400
-F 0 "C?" H 10150 5450 50  0000 R CNN
+F 0 "C11" H 10150 5450 50  0000 R CNN
 F 1 "CP100uf,10V" H 10150 5400 50  0000 R CNN
 F 2 "Capacitor_SMD:CP_Elec_6.3x5.3" H 10250 5400 50  0001 C CNN
@@
 $EndComp
 $Comp
-L taobao-c:C104,0603 C?
+L taobao-c:C104,0603 C12
 U 1 1 5CF510EC
 P 10500 5400
-F 0 "C?" H 10600 5450 50  0000 L CNN
+F 0 "C12" H 10600 5450 50  0000 L CNN
 F 1 "C104,0603" H 10600 5400 50  0000 L CNN
 F 2 "Capacitor_SMD:C_0603_1608Metric_Pad1.05x0.95mm_HandSolder" H 10500 5400 50  0001 C CNN
@@
 	10500 5200 10250 5200
 $Comp
-L power:GND #PWR?
+L power:GND #PWR0107
 U 1 1 5CF510FC
 P 10250 5600
-F 0 "#PWR?" H 10250 5350 50  0001 C CNN
+F 0 "#PWR0107" H 10250 5350 50  0001 C CNN
 F 1 "GND" H 10300 5400 50  0000 C CNN
 F 2 "" H 10250 5600 50  0001 C CNN
@@
 	10250 5500 10250 5600
 $Comp
-L power:GND #PWR?
+L power:GND #PWR0108
 U 1 1 5CF51107
 P 10500 5600
-F 0 "#PWR?" H 10500 5350 50  0001 C CNN
+F 0 "#PWR0108" H 10500 5350 50  0001 C CNN
 F 1 "GND" H 10550 5400 50  0000 C CNN
 F 2 "" H 10500 5600 50  0001 C CNN
@@
 	10750 4450 10500 4450
 $Comp
-L taobao-cp:CP100uf,10V C?
+L taobao-cp:CP100uf,10V C9
 U 1 1 5CF5EF63
 P 10250 4650
-F 0 "C?" H 10150 4700 50  0000 R CNN
+F 0 "C9" H 10150 4700 50  0000 R CNN
 F 1 "CP100uf,10V" H 10150 4650 50  0000 R CNN
 F 2 "Capacitor_SMD:CP_Elec_6.3x5.3" H 10250 4650 50  0001 C CNN
@@
 $EndComp
 $Comp
-L taobao-c:C104,0603 C?
+L taobao-c:C104,0603 C10
 U 1 1 5CF5EF6D
 P 10500 4650
-F 0 "C?" H 10600 4700 50  0000 L CNN
+F 0 "C10" H 10600 4700 50  0000 L CNN
 F 1 "C104,0603" H 10600 4650 50  0000 L CNN
 F 2 "Capacitor_SMD:C_0603_1608Metric_Pad1.05x0.95mm_HandSolder" H 10500 4650 50  0001 C CNN
@@
 	10500 4450 10250 4450
 $Comp
-L power:GND #PWR?
+L power:GND #PWR0109
 U 1 1 5CF5EF7D
 P 10250 4850
-F 0 "#PWR?" H 10250 4600 50  0001 C CNN
+F 0 "#PWR0109" H 10250 4600 50  0001 C CNN
 F 1 "GND" H 10300 4650 50  0000 C CNN
 F 2 "" H 10250 4850 50  0001 C CNN
@@
 	10250 4750 10250 4850
 $Comp
-L power:GND #PWR?
+L power:GND #PWR0110
 U 1 1 5CF5EF88
 P 10500 4850
-F 0 "#PWR?" H 10500 4600 50  0001 C CNN
+F 0 "#PWR0110" H 10500 4600 50  0001 C CNN
 F 1 "GND" H 10550 4650 50  0000 C CNN
 F 2 "" H 10500 4850 50  0001 C CNN
@@
 	10750 3650 10500 3650
 $Comp
-L taobao-cp:CP100uf,10V C?
+L taobao-cp:CP100uf,10V C7
 U 1 1 5CF5EF95
 P 10250 3850
-F 0 "C?" H 10150 3900 50  0000 R CNN
+F 0 "C7" H 10150 3900 50  0000 R CNN
 F 1 "CP100uf,10V" H 10150 3850 50  0000 R CNN
 F 2 "Capacitor_SMD:CP_Elec_6.3x5.3" H 10250 3850 50  0001 C CNN
@@
 $EndComp
 $Comp
-L taobao-c:C104,0603 C?
+L taobao-c:C104,0603 C8
 U 1 1 5CF5EF9F
 P 10500 3850
-F 0 "C?" H 10600 3900 50  0000 L CNN
+F 0 "C8" H 10600 3900 50  0000 L CNN
 F 1 "C104,0603" H 10600 3850 50  0000 L CNN
 F 2 "Capacitor_SMD:C_0603_1608Metric_Pad1.05x0.95mm_HandSolder" H 10500 3850 50  0001 C CNN
@@
 	10500 3650 10250 3650
 $Comp
-L power:GND #PWR?
+L power:GND #PWR0111
 U 1 1 5CF5EFAF
 P 10250 4050
-F 0 "#PWR?" H 10250 3800 50  0001 C CNN
+F 0 "#PWR0111" H 10250 3800 50  0001 C CNN
 F 1 "GND" H 10300 3850 50  0000 C CNN
 F 2 "" H 10250 4050 50  0001 C CNN
@@
 	10250 3950 10250 4050
 $Comp
-L power:GND #PWR?
+L power:GND #PWR0112
 U 1 1 5CF5EFBA
 P 10500 4050
-F 0 "#PWR?" H 10500 3800 50  0001 C CNN
+F 0 "#PWR0112" H 10500 3800 50  0001 C CNN
 F 1 "GND" H 10550 3850 50  0000 C CNN
 F 2 "" H 10500 4050 50  0001 C CNN

Commit message: update for rn,
Parts:
- removed RN1, RN2: R_Pack04, symbol Device:R_Pack04
- added RN? (x2): RN_103,0603, Resistor_SMD:R_Array_Concave_4x0603, symbol taobao-rpack:RN_103,0603
Connections:
- net HUB_3V3: now also RN?.5 (R4.2), RN?.6 (R3.2), RN?.7 (R2.2), RN?.8 (R1.2)
- net at U1.1 (OVCB[2]), U2.3 (FLGB): now also RN?.2 (R2.1)
- net at U1.43 (LED[1]): now also RN?.8 (R1.2)
- net at U1.44 (LED[2]): now also RN?.7 (R2.2)
- net at U1.45 (LED[3]): now also RN?.6 (R3.2)
- net at U1.46 (LED[4]): now also RN?.5 (R4.2)
- net at U1.48 (OVCB[1]), U2.2 (FLGA): now also RN?.1 (R1.1)
- net at U1.5 (OVCB[3]), U3.2 (FLGA): now also RN?.3 (R3.1)
- net at U1.7 (OVCB[4]), U3.3 (FLGB): now also RN?.4 (R4.1)
- net at D1.1 (K2), D1.2 (A2): now also RN?.1 (R1.1)
- net at D2.1 (K2), D2.2 (A2): now also RN?.2 (R2.1)
- net at D3.1 (K2), D3.2 (A2): now also RN?.3 (R3.1)
- net at D4.1 (K2), D4.2 (A2): now also RN?.4 (R4.1)
- new net: D1.1 (K2), D1.2 (A2), D2.1 (K2), D2.2 (A2), D3.1 (K2), D3.2 (A2), D4.1 (K2), D4.2 (A2), D5.2 (A), U1.42 (DRV)
Changed lines of the file:
@@
 	1    0    0    -1
 $EndComp
-$Comp
-L Device:R_Pack04 RN2
-U 1 1 5CED2755
-P 7000 4650
-F 0 "RN2" H 7200 4700 50  0000 L CNN
-F 1 "R_Pack04" H 7200 4650 50  0000 L CNN
-F 2 "" V 7275 4650 50  0001 C CNN
-F 3 "~" H 7000 4650 50  0001 C CNN
-	1    7000 4650
-	1    0    0    -1
-$EndComp
 Wire Wire Line
 	6500 4950 6800 4950
@@
 Wire Wire Line
 	9150 3850 6500 3850
-$Comp
-L Device:R_Pack04 RN1
-U 1 1 5D1966EC
-P 3750 3900
-F 0 "RN1" V 3300 3900 50  0000 C CNN
-F 1 "R_Pack04" V 3400 3900 50  0000 C CNN
-F 2 "" V 4025 3900 50  0001 C CNN
-F 3 "~" H 3750 3900 50  0001 C CNN
-	1    3750 3900
-	0    1    1    0
-$EndComp
 Connection ~ 2550 4500
 Wire Wire Line
@@
 EndData
 $EndBitmap
+$Comp
+L taobao-rpack:RN_103,0603 RN?
+U 1 1 5CEF8429
+P 3750 3900
+F 0 "RN?" V 3300 3900 50  0000 C CNN
+F 1 "RN_103,0603" V 3400 3900 50  0000 C CNN
+F 2 "Resistor_SMD:R_Array_Concave_4x0603" V 4025 3900 50  0001 C CNN
+F 3 "~" H 3750 3900 50  0001 C CNN
+	1    3750 3900
+	0    1    1    0
+$EndComp
+$Comp
+L taobao-rpack:RN_103,0603 RN?
+U 1 1 5CF10918
+P 7000 4650
+F 0 "RN?" H 7200 4700 50  0000 L CNN
+F 1 "RN_103,0603" H 7200 4650 50  0000 L CNN
+F 2 "Resistor_SMD:R_Array_Concave_4x0603" V 7275 4650 50  0001 C CNN
+F 3 "~" H 7000 4650 50  0001 C CNN
+	1    7000 4650
+	1    0    0    -1
+$EndComp
 $EndSCHEMATC
